File: Rover VCU.kicad_sch (KiCad schematic)
At the start: 6 parts, among them J3 430450400, J6 430451200

Commit message: fix: updated 12pin connector footprint + fix drc and exposed vias
Connections:
- net GND: now also J6.2 (Pin_2)
- net ESTOP: now reaches J6.8 (Pin_8)
- no-connect marks 2 -> 0
Other:
- sheet MCU ports: added ESTOP; removed none
Changed lines of the file:
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@@
 		(color 0 0 0 0)
 	)
-	(no_connect
-		(at 240.03 93.98)
-	)
-	(no_connect
-		(at 252.73 93.98)
-	)
 	(wire
 		(pts
@@
 	(wire
 		(pts
+			(xy 161.29 81.28) (xy 171.45 81.28)
+		)
+		(stroke
+			(width 0)
+			(type default)
+		)
+	)
+	(wire
+		(pts
 			(xy 77.47 40.64) (xy 77.47 43.18)
 		)
@@
 		)
 	)
+	(label "ESTOP"
+		(at 171.45 81.28 180)
+		(effects
+			(font
+				(size 1.27 1.27)
+			)
+			(justify right bottom)
+		)
+	)
+	(label "ESTOP"
+		(at 252.73 93.98 0)
+		(effects
+			(font
+				(size 1.27 1.27)
+			)
+			(justify left bottom)
+		)
+	)
 	(label "CAN2_P"
 		(at 252.73 104.14 0)
@@
 	)
 	(symbol
+		(lib_id "power:GND")
+		(at 240.03 93.98 270)
+		(mirror x)
+		(unit 1)
+		(body_style 1)
+		(exclude_from_sim no)
+		(in_bom yes)
+		(on_board yes)
+		(in_pos_files yes)
+		(dnp no)
+		(fields_autoplaced yes)
+		(property "Reference" "#PWR0103"
+			(at 233.68 93.98 0)
+			(hide yes)
+			(show_name no)
+			(do_not_autoplace no)
+			(effects
+				(font
+					(size 1.27 1.27)
+				)
+			)
+		)
+		(property "Value" "GND"
+			(at 236.22 93.9799 90)
+			(show_name no)
+			(do_not_autoplace no)
+			(effects
+				(font
+					(size 1.27 1.27)
+				)
+				(justify right)
+			)
+		)
+		(property "Footprint" ""
+			(at 240.03 93.98 0)
+			(hide yes)
+			(show_name no)
+			(do_not_autoplace no)
+			(effects
+				(font
+					(size 1.27 1.27)
+				)
+			)
+		)
+		(property "Datasheet" ""
+			(at 240.03 93.98 0)
+			(hide yes)
+			(show_name no)
+			(do_not_autoplace no)
+			(effects
+				(font
+					(size 1.27 1.27)
+				)
+			)
+		)
+		(property "Description" "Power symbol creates a global label with name \"GND\" , ground"
+			(at 240.03 93.98 0)
+			(hide yes)
+			(show_name no)
+			(do_not_autoplace no)
+			(effects
+				(font
+					(size 1.27 1.27)
+				)
+			)
+		)
+		(pin "1"
+		)
+		(instances
+			(project "Rover VCU"
+				(path "/33c96268-4ca2-4a73-94d6-a3ed4f27d429"
+					(reference "#PWR0103")
+					(unit 1)
+				)
+			)
+		)
+	)
+	(symbol
 		(lib_id "power:PWR_FLAG")
 		(at 86.36 43.18 270)
@@
 	)
 	(sheet
-		(at 134.62 83.82)
-		(size 26.67 43.18)
+		(at 134.62 78.74)
+		(size 26.67 48.26)
 		(exclude_from_sim no)
 		(in_bom yes)
 		(on_board yes)
 		(dnp no)
-		(fields_autoplaced yes)
 		(stroke
 			(width 0.1524)
@@
 		)
 		(property "Sheetname" "MCU"
-			(at 134.62 83.1084 0)
+			(at 134.62 78.0284 0)
 			(show_name no)
 			(do_not_autoplace no)
@@
 		)
 		(property "Sheetfile" "STM32G0B1.kicad_sch"
-			(at 134.62 127.5846 0)
+			(at 134.62 122.5046 0)
 			(show_name no)
 			(do_not_autoplace no)
@@
 			)
 		)
+		(pin "ESTOP" input
+			(at 161.29 81.28 0)
+			(effects
+				(font
+					(size 1.27 1.27)
+				)
+				(justify right)
+			)
+		)
