File: eth_phy.kicad_sch (KiCad schematic)
At the start: 20 parts, among them J3 Conn_01x02, U3 DP83TC812RRHARQ1

Commit message: feat: added can bus channels and psu
Parts:
- removed J3: Conn_01x02, symbol Connector_Generic:Conn_01x02
Connections:
- net TRD_N: now reaches C29.1
- net TRD_P: now reaches C28.2
Other:
- moved on the sheet: C15, C16, C17, C18, C19, C20, C21, C22, C23, C24, C25, C26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

Commit message: feat: added MVP routing implementation
Parts:
- U3: footprint VQFN36_RHA_TEX -> chenry-footprint-lib:VQFN36_RHA_TEX
Connections:
- net VDD_3V3: no longer C15.1, C16.1, C17.1, C18.1, C19.1, C20.1, C21.1, C22.1, C23.1, U3.11 (VDDA), U3.22 (VDDMAC), U3.34 (VDDIO), U3.7 (VSLEEP)
- net at U3.12 (TRD_P): now also FL1.2; no longer FL1.1
- net at U3.13 (TRD_M): now also FL1.1; no longer FL1.2
- net at FL1.3: now also C28.1; no longer C29.2
- net at FL1.4: now also C29.2; no longer C28.1
- new net: C17.1, C18.1, C19.1, U3.11 (VDDA)
- new net: C22.1, C23.1, U3.22 (VDDMAC)
- new net: C20.1, C21.1, U3.34 (VDDIO)
- new net: C15.1, C16.1, U3.7 (VSLEEP)
- no-connect marks 0 -> 12

Commit message: fix: cleaned up DRC and ERC's for major errors
Connections:
- net VDD_3V3: now also C15.1, C16.1, C17.1, C18.1, C19.1, C20.1, C21.1, C22.1, C23.1, U3.11 (VDDA), U3.22 (VDDMAC), U3.34 (VDDIO), U3.7 (VSLEEP)
Changed lines of the file:
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@@
 	(symbol
 		(lib_id "0_chenry_lib:VDD_3V3")
-		(at 27.94 64.77 90)
+		(at 31.75 64.77 90)
 		(unit 1)
 		(body_style 1)
@@
 		(fields_autoplaced yes)
 		(property "Reference" "#PWR040"
+			(at 35.56 64.77 0)
+			(hide yes)
+			(show_name no)
+			(do_not_autoplace no)
+			(effects
+				(font
+					(size 1.27 1.27)
+				)
+			)
+		)
+		(property "Value" "VDD_3V3"
+			(at 27.94 64.7699 90)
+			(show_name no)
+			(do_not_autoplace no)
+			(effects
+				(font
+					(size 1.27 1.27)
+				)
+				(justify left)
+			)
+		)
+		(property "Footprint" ""
 			(at 31.75 64.77 0)
 			(hide yes)
@@
 			)
 		)
-		(property "Value" "VDD_3V3"
-			(at 24.13 64.7699 90)
-			(show_name no)
-			(do_not_autoplace no)
-			(effects
-				(font
-					(size 1.27 1.27)
-				)
-				(justify left)
-			)
-		)
-		(property "Footprint" ""
-			(at 27.94 64.77 0)
-			(hide yes)
-			(show_name no)
-			(do_not_autoplace no)
-			(effects
-				(font
-					(size 1.27 1.27)
-				)
-			)
-		)
 		(property "Datasheet" ""
-			(at 27.94 64.77 0)
+			(at 31.75 64.77 0)
 			(hide yes)
 			(show_name no)
@@
 		)
 		(property "Description" "Power symbol creates a global label with name \"VDD\""
-			(at 27.94 64.77 0)
+			(at 31.75 64.77 0)
 			(hide yes)
 			(show_name no)
@@
 		)
 		(property "JLC_PN" ""
-			(at 27.94 64.77 0)
+			(at 31.75 64.77 0)
 			(hide yes)
 			(show_name no)
@@
 		)
 		(property "MFR_PN1" ""
-			(at 27.94 64.77 0)
+			(at 31.75 64.77 0)
 			(hide yes)
 			(show_name no)
@@
 		)
 		(property "MFR_PN2" ""
-			(at 27.94 64.77 0)
+			(at 31.75 64.77 0)
 			(hide yes)
 			(show_name no)
@@
 		)
 		(property "MFR_PN3" ""
-			(at 27.94 64.77 0)
+			(at 31.75 64.77 0)
 			(hide yes)
 			(show_name no)
@@
 	(symbol
 		(lib_id "0_chenry_lib:VDD_3V3")
-		(at 27.94 59.69 90)
+		(at 31.75 59.69 90)
 		(unit 1)
 		(body_style 1)
@@
 		(fields_autoplaced yes)
 		(property "Reference" "#PWR036"
+			(at 35.56 59.69 0)
+			(hide yes)
+			(show_name no)
+			(do_not_autoplace no)
+			(effects
+				(font
+					(size 1.27 1.27)
+				)
+			)
+		)
+		(property "Value" "VDD_3V3"
+			(at 27.94 59.6899 90)
+			(show_name no)
+			(do_not_autoplace no)
+			(effects
+				(font
+					(size 1.27 1.27)
+				)
+				(justify left)
+			)
+		)
+		(property "Footprint" ""
 			(at 31.75 59.69 0)
 			(hide yes)
@@
 			)
 		)
-		(property "Value" "VDD_3V3"
-			(at 24.13 59.6899 90)
-			(show_name no)
-			(do_not_autoplace no)
-			(effects
-				(font
-					(size 1.27 1.27)
-				)
-				(justify left)
-			)
-		)
-		(property "Footprint" ""
-			(at 27.94 59.69 0)
-			(hide yes)
-			(show_name no)
-			(do_not_autoplace no)
-			(effects
-				(font
-					(size 1.27 1.27)
-				)
-			)
-		)
 		(property "Datasheet" ""
-			(at 27.94 59.69 0)
+			(at 31.75 59.69 0)
 			(hide yes)
 			(show_name no)
@@
 		)
 		(property "Description" "Power symbol creates a global label with name \"VDD\""
-			(at 27.94 59.69 0)
+			(at 31.75 59.69 0)
 			(hide yes)
 			(show_name no)
@@
 		)
 		(property "JLC_PN" ""
-			(at 27.94 59.69 0)
+			(at 31.75 59.69 0)
 			(hide yes)
 			(show_name no)
@@
 		)
 		(property "MFR_PN1" ""
-			(at 27.94 59.69 0)
+			(at 31.75 59.69 0)
 			(hide yes)
 			(show_name no)
@@
 		)
 		(property "MFR_PN2" ""
-			(at 27.94 59.69 0)
+			(at 31.75 59.69 0)
 			(hide yes)
 			(show_name no)
@@
 		)
 		(property "MFR_PN3" ""
-			(at 27.94 59.69 0)
+			(at 31.75 59.69 0)
 			(hide yes)
 			(show_name no)
@@
 	(symbol
 		(lib_id "0_chenry_lib:VDD_3V3")
-		(at 27.94 62.23 90)
+		(at 31.75 62.23 90)
 		(unit 1)
 		(body_style 1)
@@
 		(fields_autoplaced yes)
 		(property "Reference" "#PWR037"
+			(at 35.56 62.23 0)
+			(hide yes)
+			(show_name no)
+			(do_not_autoplace no)
+			(effects
+				(font
+					(size 1.27 1.27)
+				)
+			)
+		)
+		(property "Value" "VDD_3V3"
+			(at 27.94 62.2299 90)
+			(show_name no)
+			(do_not_autoplace no)
+			(effects
+				(font
+					(size 1.27 1.27)
+				)
+				(justify left)
+			)
+		)
+		(property "Footprint" ""
 			(at 31.75 62.23 0)
 			(hide yes)
@@
 			)
 		)
-		(property "Value" "VDD_3V3"
-			(at 24.13 62.2299 90)
-			(show_name no)
-			(do_not_autoplace no)
-			(effects
-				(font
-					(size 1.27 1.27)
-				)
-				(justify left)
-			)
-		)
-		(property "Footprint" ""
-			(at 27.94 62.23 0)
-			(hide yes)
-			(show_name no)
-			(do_not_autoplace no)
-			(effects
-				(font
-					(size 1.27 1.27)
-				)
-			)
-		)
 		(property "Datasheet" ""
-			(at 27.94 62.23 0)
+			(at 31.75 62.23 0)
 			(hide yes)
 			(show_name no)
@@
 		)
 		(property "Description" "Power symbol creates a global label with name \"VDD\""
-			(at 27.94 62.23 0)
+			(at 31.75 62.23 0)
 			(hide yes)
 			(show_name no)
@@
 		)
 		(property "JLC_PN" ""
-			(at 27.94 62.23 0)
+			(at 31.75 62.23 0)
 			(hide yes)
 			(show_name no)
@@
 		)
 		(property "MFR_PN1" ""
-			(at 27.94 62.23 0)
+			(at 31.75 62.23 0)
 			(hide yes)
 			(show_name no)
@@
 		)
 		(property "MFR_PN2" ""
-			(at 27.94 62.23 0)
+			(at 31.75 62.23 0)
 			(hide yes)
 			(show_name no)
@@
 		)
 		(property "MFR_PN3" ""
-			(at 27.94 62.23 0)
+			(at 31.75 62.23 0)
 			(hide yes)
 			(show_name no)
@@
 	(symbol
 		(lib_id "0_chenry_lib:VDD_3V3")
-		(at 27.94 67.31 90)
+		(at 31.75 67.31 90)
 		(unit 1)
 		(body_style 1)
@@
 		(fields_autoplaced yes)
 		(property "Reference" "#PWR042"
+			(at 35.56 67.31 0)
+			(hide yes)
+			(show_name no)
+			(do_not_autoplace no)
+			(effects
+				(font
+					(size 1.27 1.27)
+				)
+			)
+		)
+		(property "Value" "VDD_3V3"
+			(at 27.94 67.3099 90)
+			(show_name no)
+			(do_not_autoplace no)
+			(effects
+				(font
+					(size 1.27 1.27)
+				)
+				(justify left)
+			)
+		)
+		(property "Footprint" ""
 			(at 31.75 67.31 0)
 			(hide yes)
@@
 			)
 		)
-		(property "Value" "VDD_3V3"
-			(at 24.13 67.3099 90)
-			(show_name no)
-			(do_not_autoplace no)
-			(effects
-				(font
-					(size 1.27 1.27)
-				)
-				(justify left)
-			)
-		)
-		(property "Footprint" ""
-			(at 27.94 67.31 0)
-			(hide yes)
-			(show_name no)
-			(do_not_autoplace no)
-			(effects
-				(font
-					(size 1.27 1.27)
-				)
-			)
-		)
 		(property "Datasheet" ""
-			(at 27.94 67.31 0)
+			(at 31.75 67.31 0)
 			(hide yes)
 			(show_name no)
@@
 		)
 		(property "Description" "Power symbol creates a global label with name \"VDD\""
-			(at 27.94 67.31 0)
+			(at 31.75 67.31 0)
 			(hide yes)
 			(show_name no)
@@
 		)
 		(property "JLC_PN" ""
-			(at 27.94 67.31 0)
+			(at 31.75 67.31 0)
 			(hide yes)
 			(show_name no)
@@
 		)
 		(property "MFR_PN1" ""
-			(at 27.94 67.31 0)
+			(at 31.75 67.31 0)
 			(hide yes)
 			(show_name no)
@@
 		)
 		(property "MFR_PN2" ""
-			(at 27.94 67.31 0)
+			(at 31.75 67.31 0)
 			(hide yes)
 			(show_name no)
@@
 		)
 		(property "MFR_PN3" ""
-			(at 27.94 67.31 0)
-			(hide yes)
-			(show_name no)
+			(at 31.75 67.31 0)
+			(hide yes)
+			(show_name no)

Commit message: fix: adde more changes from excel checklist for eth phy
Parts:
- removed R5: 10K, chenry-footprint-lib:R_0402, symbol 0_chenry_lib:R_0402_10K
- added C46: 4.7uF, chenry-footprint-lib:C_0402, symbol 0_chenry_lib:C_0402_4N7
- added C47: 1uF, chenry-footprint-lib:C_0402, symbol 0_chenry_lib:C_0402_1U
- added R14, R15: 1K, chenry-footprint-lib:R_0402, symbol 0_chenry_lib:R_0402_1K
- added R16: 100K, chenry-footprint-lib:R_0402, symbol 0_chenry_lib:R_0402_100K
- added R17, R18: 100R, chenry-footprint-lib:R_0402, symbol 0_chenry_lib:R_0402_100
- added R19, R5: 2K2, chenry-footprint-lib:R_0402, symbol 0_chenry_lib:R_0402_2K2
Connections:
- net GND: now also C46.2, C47.2, R16.2
- net NRST: now also C47.1, R19.2
- net RMII_MDIO: now also R5.2
- net TRD_N: now also R14.1
- net TRD_P: now also R15.1
- net VDD_3V3: now also U3.8 (WAKE), R19.1, R5.1
- net at C25.1, XTAL2.1: now also R18.2; no longer U3.5 (XI)
- net at C24.1, XTAL2.3: now also R17.2; no longer U3.4 (XO)
- new net: C46.1, R14.2, R15.2, R16.1
- new net: R17.1, U3.4 (XO)
- new net: R18.1, U3.5 (XI)
- no-connect marks 12 -> 11

Commit message: fix: final polishes for MFR
Parts:
- removed C16, C21: 1uF, chenry-footprint-lib:C_0402, symbol 0_chenry_lib:C_0402_1U
- added C48: 1uF, chenry-footprint-lib:C_0402, symbol 0_chenry_lib:C_0402_1U
- added FB1, FB2: 600Ohm @ 100MHz, Capacitor_SMD:C_0603_1608Metric, symbol 0_chenry_lib:BLM18KG601SH
Connections:
- net GND: now also C48.2
- net VDD_3V3: now also C48.1, FB1.1, FB2.1; no longer C15.1, C17.1, C18.1, C20.1, C22.1, C23.1, U3.11 (VDDA), U3.22 (VDDMAC), U3.34 (VDDIO), U3.7 (VSLEEP), U3.8 (WAKE)
- new net: C15.1, C22.1, C23.1, FB2.2, U3.11 (VDDA), U3.7 (VSLEEP), U3.8 (WAKE)
- new net: C17.1, C18.1, C20.1, FB1.2, U3.22 (VDDMAC), U3.34 (VDDIO)
Other:
- moved on the sheet: C15, C17, C18, C20, C22, C23

Commit message: fix: added leds to phy
Parts:
- added D7, D8: LED_RED_0603, LED_SMD:LED_0603_1608Metric, symbol 0_chenry_lib:LED_RED_0603
- added R23, R24: 5K1, chenry-footprint-lib:R_0402, symbol 0_chenry_lib:R_0402_5K1
Connections:
- net VDD_3V3: now also D7.2 (A), D8.2 (A)
- net at U3.35 (LED_0): now also R23.2
- net at U3.6 (LED_1): now also R24.2
- new net: D7.1 (K), R23.1
- new net: D8.1 (K), R24.1
- no-connect marks 11 -> 9
