File: STM32G0B1.kicad_sch (KiCad schematic)
At the start: 28 parts, among them J1 Conn_ST_STDC14, J2 USB4105-GF-A, SW1 TS-1088-AR02016, U1 STM32H563RITx, Y1 32.768kHz

Commit message: fix(eth_phy): completed revamp with lan8742a
BREAKING CHANGE:
Connections:
- net GPIO1: now reaches U1.10 (PC2)
- net GPIO0: now reaches U1.11 (PC3)
- no-connect marks 27 -> 25
Other:
- moved on the sheet: J2, R1, R2
