File: Rover VCU.kicad_pcb (KiCad board)
At the start: 4 copper layers, 86.2 x 44 mm, 99 parts, among them J1 Conn_ST_STDC14, J2 USB4105-GF-A, J3 430450400, J4 RJ45_Hanrun_HR911105A_Horizon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, J6 430451200, SW1 TS-1088-AR02016, U1 STM32H563RITx, U2 LAN8742A, U4 SN65HVD230, U5 SN65HVD230, U6 LMR51610, U7 NXE2S0505MC, U8 NCP1117-3.3_SOT223, Y1 32.768kHz

Commit message: fix(eth_phy): completed revamp with lan8742a
BREAKING CHANGE:
Parts:
- removed U7: NXE2S0505MC, Converter_DCDC:Converter_DCDC_Murata_NXExSxxxxMC_SMD
- added FB1: 600Ohm @ 100MHz, Capacitor_SMD:C_0603_1608Metric, F.Cu at (156.5, 81.8)
- added H5: MountingHole, MountingHole:MountingHole_3.2mm_M3, F.Cu at (147.0, 78.0)
- added H6: MountingHole, MountingHole:MountingHole_3.2mm_M3, F.Cu at (170.0, 99.0)
- H2, H4: footprint MountingHole:MountingHole_3.5mm -> MountingHole:MountingHole_3.2mm_M3
- moved C44 12.6 mm to (135.0, 79.0)
- moved C45 12.6 mm to (139.2, 83.8)
- moved U8 12.6 mm to (135.0, 84.0)
- moved D3 12.3 mm to (129.5, 88.2)
- moved C38 5.00 mm to (118.0, 85.8)
- moved C39 5.00 mm to (118.0, 84.8)
- moved C40 5.00 mm to (120.8, 82.0)
- moved C41 5.00 mm to (124.2, 87.5)
- moved C42 5.00 mm to (124.2, 86.0)
- moved C43 5.00 mm to (124.2, 84.2)
- moved H2 5.00 mm to (105.8, 78.0)
- moved J3 5.00 mm to (112.0, 89.0)
- moved L1 5.00 mm to (124.2, 80.8)
- moved R10 5.00 mm to (115.5, 80.0)
- moved R11 5.00 mm to (115.0, 81.5)
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Connections:
- C18 pad 1: Net-(U2-VDDIO) -> Net-(U2-VDD1A)
- C19 pad 1: Net-(U2-VDDCR) -> Net-(U2-VDD1A)
- C20 pad 1: Net-(U2-VDDCR) -> Net-(U2-VDD1A)
- C38 pad 2: GND_CHASIS -> GND
- C39 pad 2: GND_CHASIS -> GND
- C41 pad 1: Net-(U7-+VIN) -> Net-(D3-K)
- C41 pad 2: GND_CHASIS -> GND
- C42 pad 1: Net-(U7-+VIN) -> Net-(D3-K)
- C42 pad 2: GND_CHASIS -> GND
- C43 pad 1: Net-(U7-+VIN) -> Net-(D3-K)
- C43 pad 2: GND_CHASIS -> GND
- J3 pad 1: GND_CHASIS -> GND
- J3 pad 3: GND_CHASIS -> GND
- J6 pad 1: unconnected-(J6-Pin_1-Pad1) -> /GPIO1
- J6 pad 7: unconnected-(J6-Pin_7-Pad7) -> /GPIO0
- L1 pad 2: Net-(U7-+VIN) -> Net-(D3-K)
- R10 pad 2: GND_CHASIS -> GND
- R11 pad 1: Net-(U7-+VIN) -> Net-(D3-K)
- U1 pad 10: unconnected-(U1-PC2-Pad10) -> /GPIO1
- U1 pad 11: unconnected-(U1-PC3-Pad11) -> /GPIO0
- U2 pad 6: Net-(U2-VDDCR) -> Net-(U2-VDD1A)
- U2 pad 9: Net-(U2-VDDIO) -> Net-(U2-VDD1A)
- U6 pad 4: GND_CHASIS -> GND
Routing:
- net /MCU/RMII_TX_EN: track 1.33 -> 49.5 mm, vias 1 -> 2
- net /MCU/RMII_REF_CLK: track 1.43 -> 49.4 mm, vias 1 -> 2
- net /MCU/RMII_TXD0: track 1.33 -> 46.8 mm, vias 1 -> 2
- net /MCU/RMII_TXD1: track 1.32 -> 46.7 mm, vias 1 -> 2
- net /MCU/RMII_MDC: track 1.43 -> 46.4 mm, vias 1 -> 2
- net /MCU/RMII_RXD1: track 2.03 -> 46.7 mm, vias 1 -> 2
- net /MCU/RMII_RXD0: track 2.33 -> 46.6 mm, vias 1 -> 2
- net /MCU/RMII_CRS_DV: track 1.33 -> 44.6 mm, vias 1 -> 2
- net /MCU/RMII_MDIO: track 5.97 -> 46.6 mm, vias 1 -> 2
- net /GPIO1: track 0.00 -> 38.6 mm, vias 0 -> 1
- net /GPIO0: track 0.00 -> 38.3 mm, vias 0 -> 1
- net Net-(U2-LED2/~{INTSEL}): track 1.81 -> 38.4 mm
- net Net-(U2-LED1/REGOFF): track 1.31 -> 35.3 mm
- net Net-(U2-VDD1A): track 3.77 -> 34.7 mm, vias 1 -> 5
- net /MCU/NRST: track 52.8 -> 78.4 mm, vias 3 -> 4
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- removed copper zone on B.Cu, net GND_CHASIS
- removed copper zone on F.Cu, net GND_CHASIS
- removed copper zone on In1.Cu, net GND_CHASIS
- removed copper zone on In2.Cu, net GND_CHASIS
- removed copper zone on F.Cu, net Net-(U7-+VIN)
Other:
- board text added: "IO0"
- board text added: "IO1"
- board text removed: "TDN"
- board text removed: "TDP"

Commit message: fix: removed 3v3 on 1.2v lan core voltage
Connections:
- C19 pad 1: Net-(U2-VDD1A) -> Net-(U2-VDDCR)
- C20 pad 1: Net-(U2-VDD1A) -> Net-(U2-VDDCR)
- U2 pad 6: Net-(U2-VDD1A) -> Net-(U2-VDDCR)
Routing:
- net Net-(U2-VDD1A): track 34.7 -> 31.4 mm, vias 5 -> 4
- net Net-(U2-VDDCR): track 0.00 -> 2.52 mm
- net GND: vias 110 -> 112
